File: mcu.kicad_sch (KiCad schematic)
At the start: 13 parts, among them J11 Fan, J14 I2C, J2 Conn_01x05, J5 Conn_01x20, J7 Conn_01x20, Q6 MMBT3904, U4 AMS1117-5.0

Commit message: docs: add 3D renders, comprehensive README, CERN-OHL-S license, and update PCB routing
Parts:
- added C33, C34: 10uF, Capacitor_SMD:C_1206_3216Metric_Pad1.33x1.80mm_HandSolder, symbol Device:C
- added U7: AMS1117-3.3, Package_TO_SOT_SMD:SOT-223-3_TabPin2, symbol Regulator_Linear:AMS1117-3.3
Connections:
- net PA11 is gone; now on net PFC_PWM: J7.8 (Pin_8)
- net PB7 is gone; now on net RELAY_INRUSH: J7.15 (Pin_15)
- net SENSE_CURRENT_80V is gone; now on net PFC_VIN: J5.10 (Pin_10)
- net SENSE_VOLTAGE_80V is gone; now on net PFC_VOUT: J5.11 (Pin_11)
- net +12V: now also C33.1, U7.3 (VI)
- net PA10: now also J2.1 (Pin_1)
- net PA8: now also J2.3 (Pin_3)
- net PA9: now also J2.2 (Pin_2)
- net PB12: now also J14.4 (Pin_4), R33.2; no longer R29.1
- net PB3: no longer J2.3 (Pin_3)
- net PB4: no longer J2.2 (Pin_2)
- net PB9: no longer J14.3 (Pin_3), R34.2
- net PFC_PWM: no longer J5.14 (Pin_14)
- net PFC_VIN: no longer J5.7 (Pin_7)
- net PFC_VOUT: no longer J5.8 (Pin_8)
- net RELAY_INRUSH: no longer J5.6 (Pin_6)
- net RELAY_ON_OFF: now also J7.16 (Pin_16); no longer J5.5 (Pin_5)
- net +3V3: now reaches J5.3 (Pin_3)
- net +3V3: now also J7.20 (Pin_20), C34.1, U7.2 (VO)
- net GND renamed GND_311V
- net GND_311V: now also C33.2, C34.2, U7.1 (GND)
- net HB_FAULT renamed PB13
- net PB13: now also J14.3 (Pin_3), R34.2
- net HB_HIGH renamed PB15
- net PB15: now also J2.5 (Pin_5)
- net HB_LOW renamed PB14
- net PB14: now also R29.1
- net PA15 renamed RESET_OC
- net RESET_OC: no longer J2.5 (Pin_5)
- net PB5 renamed ENABLE
- net ENABLE: no longer J2.1 (Pin_1)
- removed net PB8: J14.4 (Pin_4), J7.16 (Pin_16), R33.2
- new net PA2: J5.14 (Pin_14)
- new net PB0: J5.8 (Pin_8)
- new net PB1: J5.7 (Pin_7)
- new net PB10: J5.6 (Pin_6)
- new net PB11: J5.5 (Pin_5)
- no-connect marks 2 -> 0
Other:
- moved on the sheet: J2, J5

Commit message: pcb: atualizar layout 2D da placa e esquematicos
Connections:
- net PA2 is gone; now on net PFC_PWM: J5.14 (Pin_14)
- net PB0 is gone; now on net PFC_VOUT: J5.8 (Pin_8)
- net PB1 is gone; now on net PFC_VIN: J5.7 (Pin_7)
- net PB10 is gone; now on net RELAY_INRUSH: J5.6 (Pin_6)
- net PB11 is gone; now on net RELAY_ON_OFF: J5.5 (Pin_5)
- net ENABLE: no longer J7.13 (Pin_13)
- net PA10: no longer J2.1 (Pin_1)
- net PA8: no longer J2.3 (Pin_3)
- net PA9: no longer J2.2 (Pin_2)
- net PB12: now also R29.1; no longer J14.4 (Pin_4), R33.2
- net PB13: no longer J14.3 (Pin_3), R34.2
- net PB14: no longer R29.1
- net PB15: no longer J2.5 (Pin_5)
- net PB3: now also J2.3 (Pin_3)
- net PB4: now also J2.2 (Pin_2)
- net PB9: now also J14.3 (Pin_3), R34.2
- net PFC_PWM: no longer J7.8 (Pin_8)
- net PFC_VIN: no longer J5.10 (Pin_10)
- net PFC_VOUT: no longer J5.11 (Pin_11)
- net RELAY_INRUSH: no longer J7.15 (Pin_15)
- net RELAY_ON_OFF: no longer J7.16 (Pin_16)
- net RESET_OC: no longer J7.10 (Pin_10)
- new net PA11: J7.8 (Pin_8)
- new net PA15: J2.5 (Pin_5), J7.10 (Pin_10)
- new net PA5: J5.11 (Pin_11)
- new net PA6: J5.10 (Pin_10)
- new net PB5: J2.1 (Pin_1), J7.13 (Pin_13)
- new net PB7: J7.15 (Pin_15)
- new net PB8: J14.4 (Pin_4), J7.16 (Pin_16), R33.2
Other:
- note added: "Isolamento do MCU? Trilha do U1C"
- note added: "PB1 -> PB6"
- note added: "PB5 -> PA11 PB4 -> PA9 PB3 -> PB15 PA15 -> PB13"
Changed lines of the file:
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@@
+		)
+	)
+	(text "Isolamento do MCU?\nTrilha do U1C\n\n"
+		(exclude_from_sim no)
+		(at 187.706 147.828 0)
+		(effects
+			(font
+				(size 1.27 1.27)
+			)
 		)
 	)
@@
 		)
 	)
+	(text "PB1 -> PB6\n"
+		(exclude_from_sim no)
+		(at 26.416 31.242 0)
+		(effects
+			(font
+				(size 1.27 1.27)
+			)
+		)
+	)
 	(text "BLACK"
 		(exclude_from_sim no)
@@
 			)
 			(justify left bottom)
+		)
+	)
+	(text " PB5 -> PA11\n PB4 -> PA9\n PB3 -> PB15\nPA15 -> PB13"
+		(exclude_from_sim no)
+		(at 121.158 173.228 0)
+		(effects
+			(font
+				(size 1.27 1.27)
+			)
+			(justify left)
 		)
 	)
@@
 		)
 	)
-	(label "PB8"
+	(label "PB11"
 		(at 34.29 24.13 0)
 		(effects
@@
 		)
 	)
-	(label "PB15"
+	(label "PA15"
 		(at 115.57 165.1 0)
 		(effects
@@
 		)
 	)
-	(label "PB12"
+	(label "PB8"
 		(at 215.9 106.68 0)
 		(effects
@@
 		)
 	)
-	(label "PA10"
+	(label "PB5"
 		(at 115.57 154.94 0)
 		(effects
@@
 		)
 	)
-	(label "PA5"
+	(label "PB0"
 		(at 34.29 34.29 0)
 		(effects
@@
 		)
 	)
-	(label "PA6"
+	(label "PB1"
 		(at 34.29 31.75 0)
 		(effects
@@
 		)
 	)
-	(label "PA8"
+	(label "PB3"
 		(at 115.57 160.02 0)
 		(effects
@@
 		)
 	)
-	(label "PA11"
+	(label "PA2"
 		(at 34.29 29.21 0)
 		(effects
@@
 		)
 	)
-	(label "PB13"
+	(label "PB9"
 		(at 215.9 109.22 0)
 		(effects
@@
 		)
 	)
-	(label "PB7"
+	(label "PB10"
 		(at 34.29 26.67 0)
-		(effects
-			(font
-				(size 1.27 1.27)
-			)
-			(justify left bottom)
-		)
-	)
-	(label "PB5"
-		(at 34.29 41.91 0)
 		(effects
 			(font
@@
 		)
 	)
-	(label "PA15"
-		(at 34.29 39.37 0)
-		(effects
-			(font
-				(size 1.27 1.27)
-			)
-			(justify left bottom)
-		)
-	)
 	(label "PA5"
 		(at 59.69 154.94 0)
@@
 		)
 	)
-	(label "PA9"
+	(label "PB4"
 		(at 115.57 157.48 0)
 		(effects
@@
 		)
 	)
-	(label "PB14"
+	(label "PB12"
 		(at 26.67 99.06 0)
 		(effects
